Commit message: complete mobile robot

File: tf-urdf-gazebo_ws/src/my_robot.urdf (robot description, URDF)
Before this commit: robot popat, 3 links, 2 joints
Links:
- removed link second_link
- removed link third_link
- added link base_footprint
- added link caster_wheel; visual sphere radius=0.05
- added link left_wheel_link; visual cylinder length=0.05 radius=0.1
- added link right_wheel_link; visual cylinder length=0.05 radius=0.1
Joints:
- removed joint joint1
- removed joint joint2
- added joint base_to_base_footprint: type fixed, parent base_link, child base_footprint, origin xyz=0 0 -0.1 rpy=0 0 0
- added joint base_to_caster_wheel: type continuous, parent base_link, child caster_wheel, origin xyz=0.2 0 -0.05 rpy=0 0 0, axis 0 0 1
- added joint base_to_left_wheel: type continuous, parent base_link, child left_wheel_link, origin xyz=-0.15 0.225 0 rpy=-1.57 0 0, axis 0 0 1
- added joint base_to_right_wheel: type continuous, parent base_link, child right_wheel_link, origin xyz=-0.15 -0.225 0 rpy=1.57 0 0, axis 0 0 1
